Commit message: Replace with a new holder to hold Straight Torch, RealSense Camera, and Keyence Scanner

File: src/roboweld_support/urdf/roboweldKeyence.xacro (robot description, xacro)
@@ -19,10 +19,29 @@
      2. The Welding table, our robot arm is installed on it.
      3. The Kinect V2, RGBD camera provides the point clouds that we need.
-     4. The UR5, our robot arm, with the Keyence LJ 7200 as its end effector.
+     4. The UR5, our robot arm, with the Straight Fronius Torch as its end effector.
+     5. The Keyence LJ7200 Laser Scanner attached to the torch holder.
+     6. The RealSense D435i attached to the torch holder.
 -->
   <!-- defining tool -->
-  <!-- Keyence LJ 7200 -->
+  <!-- Welding torch holder with the Straight Torch -->
   <xacro:property name="ref_dist_a" value="0.2"/>
-  <link name="tool0">  <!-- Actually this is LJ7200 -->
+  <link name="tool0">  <!-- Actually this is the Fronius Straight Torch held by the holder -->
+      <visual>
+        <geometry>
+          <mesh filename="package://roboweld_support/meshes/collision/STorchRCamKScan.stl"
+                scale="0.001 0.001 0.001"/>
+        </geometry>
+          <origin xyz="0 0 0" rpy="0 ${pi} 0"/>
+      </visual>
+      <collision>
+        <geometry>
+          <mesh filename="package://roboweld_support/meshes/collision/STorchRCamKScan.stl"
+                scale="0.001 0.001 0.001"/>
+        </geometry>
+          <origin xyz="0 0 0" rpy="0 ${pi} 0"/>
+      </collision>
+  </link>
+<!--
+  <link name="lj_7200">
     <visual>
       <origin xyz="0 0 0" rpy="0 0 0"/>
@@ -49,14 +68,19 @@
       <child link="tool0"/>
     </joint>
-  <!-- Optical frame -->
+-->
+  <!-- Optical frame
   <link name="lj_v7200_optical_frame"/>
   <joint name="optical_frame" type="fixed">
-  <!--
     <origin xyz="0 0 -${ref_dist_a}" rpy="0 0 0"/>
-  -->
     <origin xyz="0 0 -0.05" rpy="0 0 0"/>
     <parent link="tool0"/>
     <child link="lj_v7200_optical_frame"/>
   </joint>
+-->
+    <joint name="wrist_3_link-tool0_fixed_joint" type="fixed">
+      <origin xyz="0 -0.105 0.360" rpy="0 0 ${pi}"/>
+      <parent link="wrist_3_link"/>
+      <child link="tool0"/>
+    </joint>
   <xacro:include filename="$(find kinect2_description)/urdf/kinect2_urdf.xacro" />
   <xacro:kinect2 prefix=""/>

Commit message: Fixed the Realsense Camera position on the New Holder

File: src/roboweld_support/urdf/roboweldKeyence.xacro (robot description, xacro)
@@ -83,4 +83,32 @@
       <child link="tool0"/>
     </joint>
+  <!-- This is the link for the tail cable of the torch -->
+  <link name="tail" >
+    <visual>
+       <geometry>
+         <cylinder length="0.1" radius="0.0125"/>
+       </geometry>
+       <origin rpy="0 0 0" xyz="0 0 0"/>
+    </visual>
+    <collision>
+       <geometry>
+         <cylinder length="0.1" radius="0.0125"/>
+       </geometry>
+       <origin rpy="0 0 0" xyz="0 0 0"/>
+    </collision>
+  </link>
+  <joint name="ee_link-tail_fixed_joint" type="fixed">
+     <origin xyz="-0.08 0 0.115" rpy="0 ${pi/2.0} 0"/>
+     <parent link="ee_link"/>
+     <child link="tail"/>
+  </joint>
+  <!-- Import the realsense D435i description -->
+  <xacro:include filename="$(find realsense2_description)/urdf/_d435.urdf.xacro" />
+  <xacro:sensor_d435 parent="ee_link" use_nominal_extrinsics="true" name="d435i">
+<!--
+    <origin xyz="0.16026 0 0.01829" rpy="${pi} ${-pi} ${pi}"/>
+-->
+    <origin xyz="0.18515 0 0.0225" rpy="${pi} ${-pi} ${pi}"/>
+  </xacro:sensor_d435>
   <xacro:include filename="$(find kinect2_description)/urdf/kinect2_urdf.xacro" />
   <xacro:kinect2 prefix=""/>

Commit message: Fixed the Keyence Scanner position

File: src/roboweld_support/urdf/roboweldKeyence.xacro (robot description, xacro)
@@ -42,5 +42,4 @@
       </collision>
   </link>
-<!--
   <link name="lj_7200">
     <visual>
@@ -63,10 +62,9 @@
     </collision>
   </link>
-    <joint name="wrist_3_link-tool0_fixed_joint" type="fixed">
-      <origin xyz="0.0 0.0 0.0835" rpy="0 ${pi} ${pi/2.0}"/>
-      <parent link="wrist_3_link"/>
-      <child link="tool0"/>
-    </joint>
--->
+  <joint name="wrist_3_link-lj_7200_fixed_joint" type="fixed">
+    <origin xyz="0.062 -0.105 0.1599" rpy="0 ${pi} ${-pi/2.0}"/>
+    <parent link="wrist_3_link"/>
+    <child link="lj_7200"/>
+  </joint>
   <!-- Optical frame
   <link name="lj_v7200_optical_frame"/>

Commit message: Fixed the robot to the front of the table

File: src/roboweld_support/urdf/roboweldKeyence.xacro (robot description, xacro)
@@ -131,5 +131,5 @@
     <parent link="table"/>
     <child link="base_link"/>
-    <origin xyz="-0.6 0.0 0.015" rpy="0.0 0.0 0.0"/>
+    <origin xyz="-0.6 0.0 0.015" rpy="0.0 0.0 ${pi}"/>
   </joint>
   <!-- Optical frame -->

Commit message: Add the optical frame for the scanner

File: src/roboweld_support/urdf/roboweldKeyence.xacro (robot description, xacro)
@@ -42,5 +42,5 @@
       </collision>
   </link>
-  <link name="lj_7200">
+  <link name="lj_v7200_frame">
     <visual>
       <origin xyz="0 0 0" rpy="0 0 0"/>
@@ -62,18 +62,16 @@
     </collision>
   </link>
-  <joint name="wrist_3_link-lj_7200_fixed_joint" type="fixed">
+  <joint name="wrist_3_link-lj_v7200_fixed_joint" type="fixed">
     <origin xyz="0.062 -0.105 0.1599" rpy="0 ${pi} ${-pi/2.0}"/>
     <parent link="wrist_3_link"/>
-    <child link="lj_7200"/>
+    <child link="lj_v7200_frame"/>
   </joint>
-  <!-- Optical frame
+  <!-- Optical frame -->
   <link name="lj_v7200_optical_frame"/>
-  <joint name="optical_frame" type="fixed">
+  <joint name="optical_frame_joint" type="fixed">
     <origin xyz="0 0 -${ref_dist_a}" rpy="0 0 0"/>
-    <origin xyz="0 0 -0.05" rpy="0 0 0"/>
-    <parent link="tool0"/>
+    <parent link="lj_v7200_frame"/>
     <child link="lj_v7200_optical_frame"/>
   </joint>
--->
     <joint name="wrist_3_link-tool0_fixed_joint" type="fixed">
       <origin xyz="0 -0.105 0.360" rpy="0 0 ${pi}"/>

Commit message: Updated roboweldKeyence.xacro

File: src/roboweld_support/urdf/roboweldKeyence.xacro (robot description, xacro)
@@ -5,6 +5,80 @@
 <robot xmlns:xacro="http://ros.org/wiki/xacro"
        name="roboweld" >
+<!-- There are:-
+     1. The World, everything lives in it.
+     2. The Welding table, our robot arm is installed on it.
+     3. The Kinect V2, RGBD camera provides the point clouds that we need.
+     4. The UR5, our robot arm
+     5. The Straight Fronius Torch held by its holder
+     6. The Keyence LJ7200 Laser Scanner attached to the torch holder.
+     7. The RealSense D435i attached to the torch holder.
+-->
+<!--  1. The World, everything lives in it. -->
+  <link name="world" />
+  <joint name="world_to_table" type="fixed">
+    <parent link="world"/>
+    <child link="table"/>
+    <origin xyz="0.6 0.0 0.0" rpy="0 0 0"/>
+  </joint>
+<!-- 2. The Welding table, our robot arm is installed on it. -->
+  <link name="table">
+    <visual>
+      <geometry>
+        <box size="1.5 1.0 0.1"/>
+      </geometry>
+      <origin rpy="0 0 0" xyz="0 0 -0.05"/>
+      <material name="Steel">
+        <color rgba="1.0 0.831 0.486 1.0"/>
+      </material>
+    </visual>
+    <collision>
+      <geometry>
+        <box size="1.5 1.0 0.1"/>
+      </geometry>
+      <origin rpy="0 0 0" xyz="0 0 -0.05"/>
+    </collision>
+  </link>
+  <joint name="table_to_robot" type="fixed">
+    <parent link="table"/>
+    <child link="base_link"/>
+    <origin xyz="-0.6 0.0 0.015" rpy="0.0 0.0 ${pi}"/>
+  </joint>
+<!-- 3. The Kinect V2, RGBD camera provides the point clouds that we need.-->
+<!--    IT IS NOT USED ANYMORE -->
+<!-- We do not describe anything between the world and the camera. -->
+  <joint name="world_to_camera" type="fixed">
+    <parent link="world"/>
+    <child link="kinect2_link"/>
+<!-- Tried to calibrate the position and orientation of the camera from the World's origin -->
+<!--      <origin xyz="0.380425 0.000035 1.17336" rpy="0 3.14159 1.5707"/>
+      <origin xyz="0.050035 -0.4255 1.1515" rpy="-0.005 3.145 3.155"/>
+      <origin xyz="-0.050035 -0.4255 1.1515" rpy="-0.005 3.145 0.0134"/>
+      <origin xyz="-0.0671726 -0.438413 1.215087" rpy="-0.005 3.145 0.0134"/> -->
+      <origin xyz="0.610 0.00 1.135" rpy="3.144 -0.01 4.71"/>
+<!--      <origin xyz="0.380425 0.000035 1.17336" rpy="-2.9554254 0.1372145 1.5570305"/> -->
+  </joint>
+<!-- The Kinect V2 camera body. -->
+  <xacro:include filename="$(find kinect2_description)/urdf/kinect2_urdf.xacro" />
+  <xacro:kinect2 prefix=""/>
+  <!-- Optical frame -->
+  <link name="kinect2_rgb_optical_frame"/>
+  <joint name="rgb_optical_frame" type="fixed">
+    <origin xyz="0 0 0" rpy="0 0 0"/>
+    <parent link="kinect2_link"/> <!-- This link is defined in the kinect2_urdf.xacro file. -->
+    <child link="kinect2_rgb_optical_frame"/>
+  </joint>
+    <link name="kinect2_ir_optical_frame"/>
+    <joint name="kinect2_rgb_joint" type="fixed">
+<!--
+      <origin xyz="-0.0517134766043 0.000128911761804 0.000705039229472" rpy="0.00257173763296 -0.00373970390715 0.00528936886629"/>
+-->
+      <origin xyz="-0.0495134766043 0.000128911761804 0.0" rpy="0.00257173763296 -0.00373970390715 0.00528936886629"/>
+      <parent link="kinect2_rgb_optical_frame"/>
+      <child link="kinect2_ir_optical_frame"/>
+    </joint>
+<!-- 4. The UR5, our robot arm -->
+<!-- The Hardware Interface to the UR5 -->
   <xacro:arg name="transmission_hw_interface" default="hardware_interface/PositionJointInterface"/>
-  <!-- ur5 -->
+  <!-- ur5 body description-->
   <xacro:include filename="$(find ur_description)/urdf/ur5.urdf.xacro" />
   <!-- arm -->
@@ -14,13 +88,5 @@
     kinematics_file="${xacro.load_yaml('$(arg kinematics_config)')}"
   />
-  <link name="world" />
-<!-- There are:-
-     1. The World, everything lives in it.
-     2. The Welding table, our robot arm is installed on it.
-     3. The Kinect V2, RGBD camera provides the point clouds that we need.
-     4. The UR5, our robot arm, with the Straight Fronius Torch as its end effector.
-     5. The Keyence LJ7200 Laser Scanner attached to the torch holder.
-     6. The RealSense D435i attached to the torch holder.
--->
+<!-- The Straight Fronius Torch held by its holder -->
   <!-- defining tool -->
   <!-- Welding torch holder with the Straight Torch -->
@@ -107,59 +173,3 @@
     <origin xyz="0.18515 0 0.0225" rpy="${pi} ${-pi} ${pi}"/>
   </xacro:sensor_d435>
-  <xacro:include filename="$(find kinect2_description)/urdf/kinect2_urdf.xacro" />
-  <xacro:kinect2 prefix=""/>
-  <link name="table">
-    <visual>
-      <geometry>
-        <box size="1.5 1.0 0.1"/>
-      </geometry>
-      <origin rpy="0 0 0" xyz="0 0 -0.05"/>
-      <material name="Steel">
-        <color rgba="1.0 0.831 0.486 1.0"/>
-      </material>
-    </visual>
-    <collision>
-      <geometry>
-        <box size="1.5 1.0 0.1"/>
-      </geometry>
-      <origin rpy="0 0 0" xyz="0 0 -0.05"/>
-    </collision>
-  </link>
-  <joint name="table_to_robot" type="fixed">
-    <parent link="table"/>
-    <child link="base_link"/>
-    <origin xyz="-0.6 0.0 0.015" rpy="0.0 0.0 ${pi}"/>
-  </joint>
-  <!-- Optical frame -->
-  <link name="kinect2_rgb_optical_frame"/>
-  <joint name="rgb_optical_frame" type="fixed">
-    <origin xyz="0 0 0" rpy="0 0 0"/>
-    <parent link="kinect2_link"/> <!-- This link is defined in the kinect2_urdf.xacro file. -->
-    <child link="kinect2_rgb_optical_frame"/>
-  </joint>
-    <link name="kinect2_ir_optical_frame"/>
-    <joint name="kinect2_rgb_joint" type="fixed">
-<!--
-      <origin xyz="-0.0517134766043 0.000128911761804 0.000705039229472" rpy="0.00257173763296 -0.00373970390715 0.00528936886629"/>
--->
-      <origin xyz="-0.0495134766043 0.000128911761804 0.0" rpy="0.00257173763296 -0.00373970390715 0.00528936886629"/>
-      <parent link="kinect2_rgb_optical_frame"/>
-      <child link="kinect2_ir_optical_frame"/>
-    </joint>
-  <joint name="world_to_table" type="fixed">
-    <parent link="world"/>
-    <child link="table"/>
-    <origin xyz="0.6 0.0 0.0" rpy="0 0 0"/>
-  </joint>
-<!-- We do not describe anything between the world and the camera. -->
-  <joint name="world_to_camera" type="fixed">
-    <parent link="world"/>
-    <child link="kinect2_link"/>
-<!--      <origin xyz="0.380425 0.000035 1.17336" rpy="0 3.14159 1.5707"/>
-      <origin xyz="0.050035 -0.4255 1.1515" rpy="-0.005 3.145 3.155"/>
-      <origin xyz="-0.050035 -0.4255 1.1515" rpy="-0.005 3.145 0.0134"/>
-      <origin xyz="-0.0671726 -0.438413 1.215087" rpy="-0.005 3.145 0.0134"/> -->
-      <origin xyz="0.610 0.00 1.135" rpy="3.144 -0.01 4.71"/>
-<!--      <origin xyz="0.380425 0.000035 1.17336" rpy="-2.9554254 0.1372145 1.5570305"/> -->
-  </joint>
 </robot>

Commit message: roboweldKeyence.xacro comment explained changes

File: src/roboweld_support/urdf/roboweldKeyence.xacro (robot description, xacro)
@@ -1,5 +1,15 @@
 <?xml version="1.0"?>
 <!--
-  The xacro file for the UR5 holding the Keyence LJ7200 laser scanner as End Effector
+  The xacro file for the UR5 holding the Keyence LJ V7200 laser scanner
+  It was created by:
+  Victor W H Wu, on
+  11 May 2022.
+  For:
+  The Chinese National Engineering Research Centre for Steel Construction
+  (Hong Kong Branch)   Robotic Welding Division
+  NOTE: This version the Laser Scanner is pointing at the workpiece in the same
+  ====
+  direction as the Straight Welding Torch. There should be another version that
+  points the Laser Scanner to the workpiece at 27 degree from the Torch.
 -->
 <robot xmlns:xacro="http://ros.org/wiki/xacro"
@@ -138,37 +148,6 @@
     <child link="lj_v7200_frame"/>
   </joint>
-  <xacro:property name="ref_dist_a" value="0.2"/>
-<!--
   <xacro:include filename="$(find keyence_experimental)/urdf/lj_v7200_macro.xacro"/>
   <xacro:lj_v7200 prefix=""/>
--->
-  <link name="lj_v7200_frame">
-    <visual>
-      <origin xyz="0 0 0" rpy="0 0 0"/>
-      <geometry>
-        <mesh filename="package://keyence_experimental/meshes/visual/lj_v7200.dae"/>
-      </geometry>
-      <material name="dark grey">
-        <color rgba="0.2 0.2 0.2 1"/>
-      </material>
-    </visual>
-    <collision>
-      <origin xyz="0 0 0" rpy="0 0 0"/>
-      <geometry>
-        <mesh filename="package://keyence_experimental/meshes/collision/lj_v7200.stl"/>
-      </geometry>
-      <material name="dark grey">
-        <color rgba="0.2 0.2 0.2 1"/>
-      </material>
-    </collision>
-  </link>
-<!--
-  <link name="lj_v7200_optical_frame"/>
-  <joint name="optical_frame_joint" type="fixed">
-    <origin xyz="0 0 -${ref_dist_a}" rpy="0 0 0"/>
-    <parent link="lj_v7200_frame"/>
-    <child link="lj_v7200_optical_frame"/>
-  </joint>
--->
 <!-- 7. The RealSense D435i attached to the torch holder. NOT IN USE-->
 <!-- Import the realsense D435i description -->
