Commit message: Restore base correction to pi

File: src/fmauch_universal_robot/ur_description/urdf/ur5.urdf.xacro (robot description, xacro)
@@ -43,8 +43,8 @@
     <xacro:property name="upper_arm_inertia_offset" value="0.136" />  <!-- measured from model -->
     <!-- This is for compatibility reasons, as transformation between base and base_link was always 180 degree in the ur_description -->
+    <xacro:property name="base_correction" value="${pi}" />
     <!--
-    <xacro:property name="base_correction" value="${pi}" />
+    <xacro:property name="base_correction" value="0" />
     -->
-    <xacro:property name="base_correction" value="0" />
     <link name="${prefix}base_link" >
       <visual>

Commit message: libsocket and kinect2 description added

File: src/fmauch_universal_robot/ur_description/urdf/ur5.urdf.xacro (robot description, xacro)
@@ -23,5 +23,5 @@
     safety_k_position:=20
     kinematics_file">
-    <xacro:property name="__kinematics" value="${kinematics_file['kinematics']}"/>
+    <xacro:property name="kinematics" value="${kinematics_file['kinematics']}"/>
     <!-- Inertia parameters -->
     <xacro:property name="base_mass" value="4.0" />  <!-- This mass might be incorrect -->
@@ -70,5 +70,5 @@
       <parent link="${prefix}base_link" />
       <child link = "${prefix}shoulder_link" />
-      <origin xyz="${__kinematics['shoulder']['x']} ${__kinematics['shoulder']['y']} ${__kinematics['shoulder']['z']}" rpy="${__kinematics['shoulder']['roll']} ${__kinematics['shoulder']['pitch']} ${__kinematics['shoulder']['yaw'] + base_correction}" />
+      <origin xyz="${kinematics['shoulder']['x']} ${kinematics['shoulder']['y']} ${kinematics['shoulder']['z']}" rpy="${kinematics['shoulder']['roll']} ${kinematics['shoulder']['pitch']} ${kinematics['shoulder']['yaw'] + base_correction}" />
       <axis xyz="0 0 1" />
       <xacro:unless value="${joint_limited}">
@@ -109,5 +109,5 @@
       <parent link="${prefix}shoulder_link" />
       <child link = "${prefix}upper_arm_link" />
-      <origin xyz="${__kinematics['upper_arm']['x']} ${__kinematics['upper_arm']['y']} ${__kinematics['upper_arm']['z']}" rpy="${__kinematics['upper_arm']['roll']} ${__kinematics['upper_arm']['pitch']} ${__kinematics['upper_arm']['yaw']}" />
+      <origin xyz="${kinematics['upper_arm']['x']} ${kinematics['upper_arm']['y']} ${kinematics['upper_arm']['z']}" rpy="${kinematics['upper_arm']['roll']} ${kinematics['upper_arm']['pitch']} ${kinematics['upper_arm']['yaw']}" />
       <axis xyz="0 0 1" />
       <xacro:unless value="${joint_limited}">
@@ -141,6 +141,6 @@
         </geometry>
       </collision>
-      <xacro:cylinder_inertial radius="0.06" length="${-1*__kinematics['forearm']['x']}" mass="${upper_arm_mass}">
-        <origin xyz="${0.5*__kinematics['forearm']['x']} 0.0 ${upper_arm_inertia_offset}" rpy="0 ${pi/2} 0" />
+      <xacro:cylinder_inertial radius="0.06" length="${-1*kinematics['forearm']['x']}" mass="${upper_arm_mass}">
+        <origin xyz="${0.5*kinematics['forearm']['x']} 0.0 ${upper_arm_inertia_offset}" rpy="0 ${pi/2} 0" />
       </xacro:cylinder_inertial>
     </link>
@@ -148,5 +148,5 @@
       <parent link="${prefix}upper_arm_link" />
       <child link = "${prefix}forearm_link" />
-      <origin xyz="${__kinematics['forearm']['x']} ${__kinematics['forearm']['y']} ${__kinematics['forearm']['z']}" rpy="${__kinematics['forearm']['roll']} ${__kinematics['forearm']['pitch']} ${__kinematics['forearm']['yaw']}" />
+      <origin xyz="${kinematics['forearm']['x']} ${kinematics['forearm']['y']} ${kinematics['forearm']['z']}" rpy="${kinematics['forearm']['roll']} ${kinematics['forearm']['pitch']} ${kinematics['forearm']['yaw']}" />
       <axis xyz="0 0 1" />
       <xacro:unless value="${joint_limited}">
@@ -180,6 +180,6 @@
         </geometry>
       </collision>
-      <xacro:cylinder_inertial radius="0.06" length="${-1*__kinematics['wrist_1']['x']}" mass="${forearm_mass}">
-        <origin xyz="${0.5*__kinematics['forearm']['x']} 0.0 ${elbow_offset}" rpy="0 ${pi/2} 0" />
+      <xacro:cylinder_inertial radius="0.06" length="${-1*kinematics['wrist_1']['x']}" mass="${forearm_mass}">
+        <origin xyz="${0.5*kinematics['forearm']['x']} 0.0 ${elbow_offset}" rpy="0 ${pi/2} 0" />
       </xacro:cylinder_inertial>
     </link>
@@ -187,5 +187,5 @@
       <parent link="${prefix}forearm_link" />
       <child link = "${prefix}wrist_1_link" />
-      <origin xyz="${__kinematics['wrist_1']['x']} ${__kinematics['wrist_1']['y']} ${__kinematics['wrist_1']['z']}" rpy="${__kinematics['wrist_1']['roll']} ${__kinematics['wrist_1']['pitch']} ${__kinematics['wrist_1']['yaw']}" />
+      <origin xyz="${kinematics['wrist_1']['x']} ${kinematics['wrist_1']['y']} ${kinematics['wrist_1']['z']}" rpy="${kinematics['wrist_1']['roll']} ${kinematics['wrist_1']['pitch']} ${kinematics['wrist_1']['yaw']}" />
       <axis xyz="0 0 1" />
       <xacro:unless value="${joint_limited}">
@@ -219,5 +219,5 @@
         </geometry>
       </collision>
-      <xacro:cylinder_inertial radius="0.075" length="${-1*__kinematics['wrist_2']['y']}" mass="${wrist_1_mass}">
+      <xacro:cylinder_inertial radius="0.075" length="${-1*kinematics['wrist_2']['y']}" mass="${wrist_1_mass}">
         <origin xyz="0.0 0.0 0.0" rpy="0 0 0" />
       </xacro:cylinder_inertial>
@@ -226,5 +226,5 @@
       <parent link="${prefix}wrist_1_link" />
       <child link = "${prefix}wrist_2_link" />
-      <origin xyz="${__kinematics['wrist_2']['x']} ${__kinematics['wrist_2']['y']} ${__kinematics['wrist_2']['z']}" rpy="${__kinematics['wrist_2']['roll']} ${__kinematics['wrist_2']['pitch']} ${__kinematics['wrist_2']['yaw']}" />
+      <origin xyz="${kinematics['wrist_2']['x']} ${kinematics['wrist_2']['y']} ${kinematics['wrist_2']['z']}" rpy="${kinematics['wrist_2']['roll']} ${kinematics['wrist_2']['pitch']} ${kinematics['wrist_2']['yaw']}" />
       <axis xyz="0 0 1" />
       <xacro:unless value="${joint_limited}">
@@ -258,5 +258,5 @@
         </geometry>
       </collision>
-      <xacro:cylinder_inertial radius="0.06" length="${__kinematics['wrist_3']['y']}" mass="${wrist_2_mass}">
+      <xacro:cylinder_inertial radius="0.06" length="${kinematics['wrist_3']['y']}" mass="${wrist_2_mass}">
         <origin xyz="0.0 0.0 0.0" rpy="0 0 0" />
       </xacro:cylinder_inertial>
@@ -265,5 +265,5 @@
       <parent link="${prefix}wrist_2_link" />
       <child link = "${prefix}wrist_3_link" />
-      <origin xyz="${__kinematics['wrist_3']['x']} ${__kinematics['wrist_3']['y']} ${__kinematics['wrist_3']['z']}" rpy="${__kinematics['wrist_3']['roll']} ${__kinematics['wrist_3']['pitch']} ${__kinematics['wrist_3']['yaw']}" />
+      <origin xyz="${kinematics['wrist_3']['x']} ${kinematics['wrist_3']['y']} ${kinematics['wrist_3']['z']}" rpy="${kinematics['wrist_3']['roll']} ${kinematics['wrist_3']['pitch']} ${kinematics['wrist_3']['yaw']}" />
       <axis xyz="0 0 1" />
       <xacro:unless value="${joint_limited}">

File: src/roboweld_support/urdf/roboweldKeyence.xacro (robot description, xacro)
@@ -12,5 +12,5 @@
   <xacro:ur5_robot prefix="" joint_limited="true"
     transmission_hw_interface="$(arg transmission_hw_interface)"
-    kinematics_file="${load_yaml('$(arg kinematics_config)')}"
+    kinematics_file="${xacro.load_yaml('$(arg kinematics_config)')}"
   />
   <link name="world" />
