Commit message: Keyence lj_v7200_macro.xacro modified

File: src/keyence_experimental/urdf/lj_v7200_macro.xacro (robot description, xacro)
@@ -24,9 +24,10 @@
     </link>
     <!-- Optical frame -->
+<!-- The parent and child of this joint was swapped by Victor Wu on 11 May 2022. -->
     <link name="${prefix}lj_v7200_optical_frame"/>
     <joint name="optical_frame" type="fixed">
       <origin xyz="0 0 ${ref_dist_a}" rpy="0 0 0"/>
-      <parent link="${prefix}lj_v7200_optical_frame"/>
-      <child link="${prefix}lj_v7200_frame"/>
+      <child link="${prefix}lj_v7200_optical_frame"/>
+      <parent link="${prefix}lj_v7200_frame"/>
    </joint>
   </xacro:macro>

File: src/roboweld_support/urdf/roboweldKeyence.xacro (robot description, xacro)
@@ -8,9 +8,9 @@
      1. The World, everything lives in it.
      2. The Welding table, our robot arm is installed on it.
-     3. The Kinect V2, RGBD camera provides the point clouds that we need.
+     3. The Kinect V2, RGBD camera provides the point clouds that we need. NOT IN USE ANYMORE
      4. The UR5, our robot arm
      5. The Straight Fronius Torch held by its holder
      6. The Keyence LJ7200 Laser Scanner attached to the torch holder.
-     7. The RealSense D435i attached to the torch holder.
+     7. The RealSense D435i attached to the torch holder. NOT IN USE
 -->
 <!--  1. The World, everything lives in it. -->
@@ -88,9 +88,13 @@
     kinematics_file="${xacro.load_yaml('$(arg kinematics_config)')}"
   />
-<!-- The Straight Fronius Torch held by its holder -->
-  <!-- defining tool -->
+<!-- 5. The Straight Fronius Torch held by its holder-->
   <!-- Welding torch holder with the Straight Torch -->
-  <xacro:property name="ref_dist_a" value="0.2"/>
-  <link name="tool0">  <!-- Actually this is the Fronius Straight Torch held by the holder -->
+  <joint name="wrist_3_link-tool0_fixed_joint" type="fixed">
+    <origin xyz="0 -0.105 0.360" rpy="0 0 ${pi}"/>
+    <parent link="wrist_3_link"/>
+    <child link="tool0"/>
+  </joint>
+  <!-- Actually this is the Fronius Straight Torch held by the holder -->
+    <link name="tool0">
       <visual>
         <geometry>
@@ -108,4 +112,35 @@
       </collision>
   </link>
+  <joint name="ee_link-tail_fixed_joint" type="fixed">
+     <origin xyz="-0.08 0 0.115" rpy="0 ${pi/2.0} 0"/>
+     <parent link="ee_link"/>
+     <child link="tail"/>
+  </joint>
+  <!-- This is the link for the tail cable of the torch -->
+  <link name="tail" >
+    <visual>
+       <geometry>
+         <cylinder length="0.1" radius="0.0125"/>
+       </geometry>
+       <origin rpy="0 0 0" xyz="0 0 0"/>
+    </visual>
+    <collision>
+       <geometry>
+         <cylinder length="0.1" radius="0.0125"/>
+       </geometry>
+       <origin rpy="0 0 0" xyz="0 0 0"/>
+    </collision>
+  </link>
+<!-- 6. The Keyence LJ7200 Laser Scanner attached to the torch holder. -->
+  <joint name="wrist_3_link-lj_v7200_fixed_joint" type="fixed">
+    <origin xyz="0.062 -0.105 0.1599" rpy="0 ${pi} ${-pi/2.0}"/>
+    <parent link="wrist_3_link"/>
+    <child link="lj_v7200_frame"/>
+  </joint>
+  <xacro:property name="ref_dist_a" value="0.2"/>
+<!--
+  <xacro:include filename="$(find keyence_experimental)/urdf/lj_v7200_macro.xacro"/>
+  <xacro:lj_v7200 prefix=""/>
+-->
   <link name="lj_v7200_frame">
     <visual>
@@ -128,10 +163,5 @@
     </collision>
   </link>
-  <joint name="wrist_3_link-lj_v7200_fixed_joint" type="fixed">
-    <origin xyz="0.062 -0.105 0.1599" rpy="0 ${pi} ${-pi/2.0}"/>
-    <parent link="wrist_3_link"/>
-    <child link="lj_v7200_frame"/>
-  </joint>
-  <!-- Optical frame -->
+<!--
   <link name="lj_v7200_optical_frame"/>
   <joint name="optical_frame_joint" type="fixed">
@@ -140,35 +170,9 @@
     <child link="lj_v7200_optical_frame"/>
   </joint>
-    <joint name="wrist_3_link-tool0_fixed_joint" type="fixed">
-      <origin xyz="0 -0.105 0.360" rpy="0 0 ${pi}"/>
-      <parent link="wrist_3_link"/>
-      <child link="tool0"/>
-    </joint>
-  <!-- This is the link for the tail cable of the torch -->
-  <link name="tail" >
-    <visual>
-       <geometry>
-         <cylinder length="0.1" radius="0.0125"/>
-       </geometry>
-       <origin rpy="0 0 0" xyz="0 0 0"/>
-    </visual>
-    <collision>
-       <geometry>
-         <cylinder length="0.1" radius="0.0125"/>
-       </geometry>
-       <origin rpy="0 0 0" xyz="0 0 0"/>
-    </collision>
-  </link>
-  <joint name="ee_link-tail_fixed_joint" type="fixed">
-     <origin xyz="-0.08 0 0.115" rpy="0 ${pi/2.0} 0"/>
-     <parent link="ee_link"/>
-     <child link="tail"/>
-  </joint>
-  <!-- Import the realsense D435i description -->
+-->
+<!-- 7. The RealSense D435i attached to the torch holder. NOT IN USE-->
+<!-- Import the realsense D435i description -->
   <xacro:include filename="$(find realsense2_description)/urdf/_d435.urdf.xacro" />
   <xacro:sensor_d435 parent="ee_link" use_nominal_extrinsics="true" name="d435i">
-<!--
-    <origin xyz="0.16026 0 0.01829" rpy="${pi} ${-pi} ${pi}"/>
--->
     <origin xyz="0.18515 0 0.0225" rpy="${pi} ${-pi} ${pi}"/>
   </xacro:sensor_d435>

Commit message: Updates just before demo

File: src/keyence_experimental/urdf/lj_v7200_macro.xacro (robot description, xacro)
@@ -28,6 +28,6 @@
     <joint name="optical_frame" type="fixed">
       <origin xyz="0 0 ${ref_dist_a}" rpy="0 0 0"/>
-      <child link="${prefix}lj_v7200_optical_frame"/>
-      <parent link="${prefix}lj_v7200_frame"/>
+      <parent link="${prefix}lj_v7200_optical_frame"/>
+      <child link="${prefix}lj_v7200_frame"/>
    </joint>
   </xacro:macro>

File: src/roboweld_support/urdf/roboweldtilkey.xacro (robot description, xacro)
@@ -145,7 +145,7 @@
 <!-- 6. The Keyence LJ7200 Laser Scanner attached to the torch holder. -->
   <joint name="wrist_3_link-lj_v7200_fixed_joint" type="fixed">
-    <origin xyz="0.11692 -0.105 0.18224" rpy="-0.471238898038469 ${pi} ${-pi/2.0}"/> <!-- for tilted scanner -->
+    <origin xyz="0.00433 -0.105 0.350441" rpy="-0.471238898038469 ${pi} ${-pi/2.0}"/> <!-- for tilted scanner -->
     <parent link="wrist_3_link"/>
-    <child link="lj_v7200_frame"/>
+    <child link="lj_v7200_optical_frame"/>
   </joint>
   <xacro:include filename="$(find keyence_experimental)/urdf/lj_v7200_macro.xacro"/>

Commit message: some updates

File: src/keyence_experimental/urdf/lj_v7200_macro.xacro (robot description, xacro)
@@ -30,5 +30,5 @@
       <parent link="${prefix}lj_v7200_optical_frame"/>
       <child link="${prefix}lj_v7200_frame"/>
-   </joint>
+    </joint>
   </xacro:macro>
 </robot>
